Commit message: adding camera and lidar sensors

File: go_chase_it/urdf/robot.xacro (robot description, xacro)
@@ -116,3 +116,63 @@
 		<dynamics damping="1.0" friction="1.0"/>
 	</joint>
+	<!--Camera Sensor-->
+	<link name="camera">
+		<pose>0 0 0 0 0 0</pose>
+		<inertial>
+			<mass value="0.1"/>
+			<origin xyz="0 0 0" rpy=" 0 0 0"/>
+			<inertia
+		ixx="1e-6" ixy="0" ixz="0"
+		iyy="1e-6" iyz="0" izz="1e-6"
+	/>
+		</inertial>
+		<collision>
+			<origin xyz="0 0 0" rpy=" 0 0 0"/>
+			<geometry>
+				<box size=".05 .05 .05"/>
+			</geometry>
+		</collision>
+		<visual>
+			<origin xyz="0 0 0" rpy=" 0 0 0"/>
+			<geometry>
+				<box size=".05 .05 .05"/>
+			</geometry>
+		</visual>
+	</link>
+	<joint type="fixed" name="camera_joint">
+		<origin xyz="0.2 0 0" rpy="0 0 0"/>
+		<child link="camera"/>
+		<parent link="chassis"/>
+		<axis xyz="0 1 0" rpy="0 0 0"/>
+	</joint>
+	<!--Hokuyo Lidar sensor-->
+	<link name="hokuyo">
+		<pose>0 0 0 0 0 0</pose>
+		<inertial>
+			<mass value="1e-5"/>
+			<origin xyz="0 0 0" rpy=" 0 0 0"/>
+			<inertia
+		ixx="1e-6" ixy="0" ixz="0"
+		iyy="1e-6" iyz="0" izz="1e-6"
+	/>
+		</inertial>
+		<collision>
+			<origin xyz="0 0 0" rpy=" 0 0 0"/>
+			<geometry>
+				<box size=".1 .1 .1"/>
+			</geometry>
+		</collision>
+		<visual>
+			<origin xyz="0 0 0" rpy=" 0 0 0"/>
+			<geometry>
+				<mesh filename="package://go_chase_it/meshes/hokuyo.dae"/>
+			</geometry>
+		</visual>
+	</link>
+	<joint type="fixed" name="hokuyo_joint">
+		<origin xyz="0.15 0 0.1" rpy="0 0 0"/>
+		<child link="hokuyo"/>
+		<parent link="chassis"/>
+		<axis xyz="0 1 0" rpy="0 0 0"/>
+	</joint>
 </robot>

Commit message: integrating Rviz

File: go_chase_it/urdf/robot.xacro (robot description, xacro)
@@ -1,4 +1,5 @@
 <?xml version='1.0'?>
 <robot name="my_robot" xmlns:xacro="http://www.ros.org/wiki/xacro">
+	<xacro:include filename="$(find go_chase_it)/urdf/robot.gazebo"/>
 	<link name="robot_footprint"></link>
 	<joint name="robot_footprint_joint" type="fixed">
@@ -13,7 +14,7 @@
 			<origin xyz="0.0 0 0" rpy=" 0 0 0"/>
 			<inertia
-		ixx="0.1" ixy="0" ixz="0"
-		iyy="0.1" iyz="0" izz="0.1"
-	/>
+				ixx="0.1" ixy="0" ixz="0"
+				iyy="0.1" iyz="0" izz="0.1"
+			/>
 		</inertial>
 		<collision name='collision'>
@@ -64,5 +65,5 @@
 	/>
 		</inertial>
-		<collision>
+		<collision name="left_wheel_collision">
 			<origin xyz="0 0 0" rpy=" 0 1.5707 1.5707"/>
 			<geometry>
@@ -70,5 +71,5 @@
 			</geometry>
 		</collision>
-		<visual>
+		<visual name="left_wheel_visual">
 			<origin xyz="0 0 0" rpy=" 0 1.5707 1.5707"/>
 			<geometry>
@@ -95,5 +96,5 @@
 	/>
 		</inertial>
-		<collision>
+		<collision name="right_wheel_collision">
 			<origin xyz="0 0 0" rpy=" 0 1.5707 1.5707"/>
 			<geometry>
@@ -101,5 +102,5 @@
 			</geometry>
 		</collision>
-		<visual>
+		<visual name="right_wheel_visual">
 			<origin xyz="0 0 0" rpy=" 0 1.5707 1.5707"/>
 			<geometry>
@@ -118,14 +119,13 @@
 	<!--Camera Sensor-->
 	<link name="camera">
-		<pose>0 0 0 0 0 0</pose>
 		<inertial>
 			<mass value="0.1"/>
 			<origin xyz="0 0 0" rpy=" 0 0 0"/>
 			<inertia
-		ixx="1e-6" ixy="0" ixz="0"
-		iyy="1e-6" iyz="0" izz="1e-6"
-	/>
+				ixx="1e-6" ixy="0" ixz="0"
+				iyy="1e-6" iyz="0" izz="1e-6"
+			/>
 		</inertial>
-		<collision>
+		<collision name="camera_collision">
 			<origin xyz="0 0 0" rpy=" 0 0 0"/>
 			<geometry>
@@ -133,5 +133,5 @@
 			</geometry>
 		</collision>
-		<visual>
+		<visual name="camera_visual">
 			<origin xyz="0 0 0" rpy=" 0 0 0"/>
 			<geometry>
@@ -148,14 +148,13 @@
 	<!--Hokuyo Lidar sensor-->
 	<link name="hokuyo">
-		<pose>0 0 0 0 0 0</pose>
 		<inertial>
 			<mass value="1e-5"/>
 			<origin xyz="0 0 0" rpy=" 0 0 0"/>
 			<inertia
-		ixx="1e-6" ixy="0" ixz="0"
-		iyy="1e-6" iyz="0" izz="1e-6"
-	/>
+				ixx="1e-6" ixy="0" ixz="0"
+				iyy="1e-6" iyz="0" izz="1e-6"
+			/>
 		</inertial>
-		<collision>
+		<collision name="hokuyo_collision">
 			<origin xyz="0 0 0" rpy=" 0 0 0"/>
 			<geometry>
@@ -163,5 +162,5 @@
 			</geometry>
 		</collision>
-		<visual>
+		<visual name="hokuyo_visual">
 			<origin xyz="0 0 0" rpy=" 0 0 0"/>
 			<geometry>
@@ -176,3 +175,15 @@
 		<axis xyz="0 1 0" rpy="0 0 0"/>
 	</joint>
+	<gazebo reference="chassis">
+		<material>Gazebo/Green</material>
+	</gazebo>
+	<gazebo reference="right_wheel">
+		<material>Gazebo/Blue</material>
+	</gazebo>
+	<gazebo reference="left_wheel">
+		<material>Gazebo/Blue</material>
+	</gazebo>
+	<gazebo reference="camera">
+		<material>Gazebo/Red</material>
+	</gazebo>
 </robot>

Commit message: fixing robot drive

File: go_chase_it/urdf/robot.xacro (robot description, xacro)
@@ -79,5 +79,5 @@
 	</link>
 	<joint type="continuous" name="left_wheel_hinge">
-		<origin xyz="0 -0.15 0" rpy="0 0 0"/>
+		<origin xyz="0 0.125 0" rpy="0 0 0"/>
 		<child link="left_wheel"/>
 		<parent link="chassis"/>
@@ -110,5 +110,5 @@
 	</link>
 	<joint type="continuous" name="right_wheel_hinge">
-		<origin xyz="0 0.15 0" rpy="0 0 0"/>
+		<origin xyz="0 -0.125 0" rpy="0 0 0"/>
 		<child link="right_wheel"/>
 		<parent link="chassis"/>
